Commit message: camera : C920 tete en bas, image droite et reperes coherents (phase 1)
usb_cam (MJPEG natif, mise au point fixe) publie l'image brute dans le
repere optique physique : la CAO place ce repere comme pour une camera
droite, camera.mount_rpy le retourne d'un demi-tour autour de l'axe optique
par le meme mecanisme que le LiDAR (fix_urdf generalise a toute section
frame + mount_rpy). ImageFlipNode remet l'image a l'endroit dans
camera_upright_optical_frame, declare dans l'URDF avec la meme rotation que
le TF que diffuse le noeud : pas de double parent. Le noeud ne corrige pas le
point principal, la calibration se fait donc sur /camera/image.

Regle udev sur l'index 0 seulement (l'index 1 est la metadonnee UVC),
groupe video dans install.sh, launch qui se retire sans /dev/camera, camera
Gazebo droite par construction sur les memes topics, calibration provisoire
a remplacer par la mire. Valide en simulation ; reste a faire sur le robot :
orientation optique, calibration, cout CPU.

File: alidade_description/urdf/alidade.urdf.xacro (robot description, xacro)
@@ -29,4 +29,17 @@
   <!-- Geometrie, masses et collisions : export Onshape corrige. -->
   <xacro:include filename="$(find alidade_description)/urdf/generated/alidade_${revision}.urdf"/>
+  <!-- Repere de l'image droite : la camera est montee tete en bas, son repere
+       optique (retourne par fix_urdf) decrit l'image brute ; l'image remise a
+       l'endroit par ImageFlipNode vit dans ce repere, tourne d'un demi-tour
+       autour de l'axe optique. Le noeud diffuse la meme transformation : les
+       deux sources concordent, et la simulation, qui n'a pas de noeud de
+       retournement, publie directement ici. -->
+  <xacro:property name="cam" value="${hw['camera']}"/>
+  <link name="${cam['upright_frame']}"/>
+  <joint name="${cam['upright_frame']}_joint" type="fixed">
+    <origin xyz="0 0 0" rpy="0 0 ${pi}"/>
+    <parent link="${cam['frame']}"/>
+    <child link="${cam['upright_frame']}"/>
+  </joint>
   <xacro:include filename="$(find alidade_description)/urdf/ros2_control.xacro"/>
   <xacro:alidade_ros2_control hw="${hw}" target="${target}" use_mock="${use_mock}" pico_port="$(arg pico_port)"/>

File: alidade_description/urdf/gazebo.xacro (robot description, xacro)
@@ -63,4 +63,33 @@
       </sensor>
     </gazebo>
+    <!-- Camera simulee, droite par construction : elle publie directement dans
+         le repere de l'image remise a l'endroit, sur les topics que le noeud de
+         retournement produit sur le robot reel. Le capteur Gazebo regarde le
+         long de +x de sa pose ; on le place a l'origine du repere optique,
+         qui regarde le long de +x de camera_link. -->
+    <xacro:property name="camera" value="${hw['camera']}"/>
+    <gazebo reference="camera_link">
+      <sensor name="camera" type="camera">
+        <!-- gz publie l'image sur ce topic et le camera_info a cote de lui. -->
+        <topic>camera/image</topic>
+        <update_rate>${camera['fps']}</update_rate>
+        <always_on>1</always_on>
+        <visualize>false</visualize>
+        <gz_frame_id>${camera['upright_frame']}</gz_frame_id>
+        <pose>0.0375 0 -0.0295 0 0 0</pose>
+        <camera>
+          <horizontal_fov>${camera['sim_horizontal_fov']}</horizontal_fov>
+          <image>
+            <width>${camera['width']}</width>
+            <height>${camera['height']}</height>
+            <format>R8G8B8</format>
+          </image>
+          <clip>
+            <near>0.05</near>
+            <far>10.0</far>
+          </clip>
+        </camera>
+      </sensor>
+    </gazebo>
     <!-- IMU simulee, lue par gz_ros2_control sous le nom 'imu' et publiee par
          le meme imu_sensor_broadcaster que sur le robot reel. -->

Commit message: camera : montee a l'endroit, sans noeud de retournement
La C920 est maintenant a l'endroit : le repere optique de la CAO la decrit
telle quelle. Disparaissent mount_rpy, ImageFlipNode, le repere
camera_upright_optical_frame et la dependance a image_rotate. usb_cam publie
directement /camera/image et /camera/camera_info, par une seule regle de
remappage : les consommateurs (interface, ArUco, simulation) ne changent pas
de topic, la supervision suit le camera_info.

La camera simulee etait placee par une pose recopiee a la main, perimee
avec le nouveau support. Elle est accrochee au repere optique, avec la seule
rotation de convention entre Gazebo et le repere optique : apres conversion
SDF, elle est a (115.7, 0, 102.8) mm et plonge de 25.0 degres, comme la CAO.

Un test verifie que l'image est droite et que la camera vise devant, vers le
sol : un export retourne ou un mount_rpy oublie ferait echouer le build. Le
README donne la plage utile du montage : cube entier dans l'image de 11 a
55 cm devant le chassis, avec la focale mesuree.

File: alidade_description/urdf/alidade.urdf.xacro (robot description, xacro)
@@ -29,17 +29,4 @@
   <!-- Geometrie, masses et collisions : export Onshape corrige. -->
   <xacro:include filename="$(find alidade_description)/urdf/generated/alidade_${revision}.urdf"/>
-  <!-- Repere de l'image droite : la camera est montee tete en bas, son repere
-       optique (retourne par fix_urdf) decrit l'image brute ; l'image remise a
-       l'endroit par ImageFlipNode vit dans ce repere, tourne d'un demi-tour
-       autour de l'axe optique. Le noeud diffuse la meme transformation : les
-       deux sources concordent, et la simulation, qui n'a pas de noeud de
-       retournement, publie directement ici. -->
-  <xacro:property name="cam" value="${hw['camera']}"/>
-  <link name="${cam['upright_frame']}"/>
-  <joint name="${cam['upright_frame']}_joint" type="fixed">
-    <origin xyz="0 0 0" rpy="0 0 ${pi}"/>
-    <parent link="${cam['frame']}"/>
-    <child link="${cam['upright_frame']}"/>
-  </joint>
   <xacro:include filename="$(find alidade_description)/urdf/ros2_control.xacro"/>
   <xacro:alidade_ros2_control hw="${hw}" target="${target}" use_mock="${use_mock}" pico_port="$(arg pico_port)"/>

File: alidade_description/urdf/gazebo.xacro (robot description, xacro)
@@ -63,11 +63,11 @@
       </sensor>
     </gazebo>
-    <!-- Camera simulee, droite par construction : elle publie directement dans
-         le repere de l'image remise a l'endroit, sur les topics que le noeud de
-         retournement produit sur le robot reel. Le capteur Gazebo regarde le
-         long de +x de sa pose ; on le place a l'origine du repere optique,
-         qui regarde le long de +x de camera_link. -->
+    <!-- Camera simulee, accrochee au repere optique lui-meme : sa position et
+         son inclinaison viennent de l'export, rien n'est recopie ici. Le
+         capteur Gazebo regarde le long de +x avec +z en haut, le repere optique
+         le long de +z avec +y en bas ; la pose ci-dessous passe de l'un a
+         l'autre. C'est une convention, constante quel que soit le montage. -->
     <xacro:property name="camera" value="${hw['camera']}"/>
-    <gazebo reference="camera_link">
+    <gazebo reference="${camera['frame']}">
       <sensor name="camera" type="camera">
         <!-- gz publie l'image sur ce topic et le camera_info a cote de lui. -->
@@ -76,6 +76,6 @@
         <always_on>1</always_on>
         <visualize>false</visualize>
-        <gz_frame_id>${camera['upright_frame']}</gz_frame_id>
-        <pose>0.0375 0 -0.0295 0 0 0</pose>
+        <gz_frame_id>${camera['frame']}</gz_frame_id>
+        <pose>0 0 0 ${pi/2} ${-pi/2} 0</pose>
         <camera>
           <horizontal_fov>${camera['sim_horizontal_fov']}</horizontal_fov>
