Commit message: revision v2 : chassis redessine, RealSense D435i, IMU par TF
Le robot a ete entierement refait. La v1 decrivait une machine qui n'existe
plus : elle est supprimee, pas archivee. Un seul commit parce que les quatre
volets ci-dessous sont indissociables -- separer le zero de lidar.mount_rpy du
flip_x_axis qui le compense produirait un etat intermediaire faux.

GEOMETRIE. Plateau 158x156 -> 250x252 mm, roues O64 -> O99.6, entraxe 191 ->
225 (CAO), roulette O22 a l'avant -> O50 a l'arriere, LiDAR recule de 146 mm et
monte de 11. Moteurs, reducteur, encodeurs, Pi, batterie, LiDAR et IMU sont les
MEMES pieces : volumes d'export identiques au centieme, leurs mesures sont
reprises sans reserve.

L'axe des roues n'est plus au milieu : base_footprint est a 55 mm de l'avant et
199 de l'arriere, pour un rayon circonscrit de 235 mm contre 148. Le modele
circulaire de nav2 reserve donc 18 cm de trop devant ; une empreinte polygonale
est a envisager quand la navigation reprendra.

Mesure en simulation : rayon efficace 49.998 mm pour 50.0 declares, mais
entraxe efficace 221.0 pour 225.0 -- le contact du disque de collision ne tombe
pas dans son plan median. Les roues sont ecartees de 2.0 mm, l'entraxe retombe
a 225.0 exactement, 0.0 mm d'ecart entre les deux sens.

Attention a la traction : le centre de masse passe de +26 a -90 mm, donc la
roulette non motrice porte 53 % du poids contre 27 % avant. Avec des roues 1.53
fois plus grandes, l'acceleration disponible chute d'environ un tiers.

IMU. Elle est montee A L'ENVERS et l'export le decrit fidement ; c'est
gyro_odom.py qui avait tort en lisant angular_velocity.z brut. Il ramene
desormais la vitesse angulaire dans le repere de la base par TF, la rotation
etant lue une fois et mise en cache (le joint est fixe). Sans cela : distances
justes, cap inverse -- mesure en simulation, robot tournant de +26.3 deg pour
un gyromètre annoncant -0.439 rad/s. Sept tests fixent la convention.

LIDAR. La fleche du C1 est bien le 0 du balayage (datasheet figure 1-2) et elle
est alignee sur +x : rien a corriger dans la CAO. Le demi-tour venait du
PILOTE, qui publie theta_ros = pi - theta_brut la ou la conversion juste est
-theta_brut. La correction passe donc dans rplidar.yaml (flip_x_axis: true) et
lidar.mount_rpy retombe a zero. lidar_zero.py verifie le tout au banc.

CAMERA. RealSense D435i. La geometrie interne du capteur vient de
realsense2_description, source amont : la revision n'y accroche qu'un point de
fixation, et la CAO place ce repere sur la vis, ce qui rend le decalage nul.
use_nominal_extrinsics distingue les deux cas -- en simulation la macro publie
les reperes optiques, sur le robot c'est le pilote, avec les extrinseques
CALIBREES de l'exemplaire. Meme sujet des deux cotes
(/camera/color/image_raw) : le detecteur ne sait pas ou il tourne.

Au passage, telemetry.yaml surveillait /camera/camera_info, qui n'existe plus :
la supervision aurait declare la camera morte en permanence.

Le fichier de revision porte une section `provisional` que le build rappelle a
chaque compilation : rayon, entraxe et masses sont des cotes CAO ou des pesees
de l'ancien chassis. Rien de ce qui en depend ne peut etre juge avant
`odom_calib.py`.

Co-Authored-By: Claude Opus 5 <noreply@anthropic.com>

File: alidade_description/urdf/alidade.urdf.xacro (robot description, xacro)
@@ -15,5 +15,5 @@
 -->
 <robot xmlns:xacro="http://www.ros.org/wiki/xacro" name="alidade">
-  <xacro:arg name="hardware_revision" default="v1"/>
+  <xacro:arg name="hardware_revision" default="v2"/>
   <xacro:arg name="target" default="real"/>
   <xacro:arg name="use_mock_hardware" default="false"/>
@@ -29,4 +29,17 @@
   <!-- Geometrie, masses et collisions : export Onshape corrige. -->
   <xacro:include filename="$(find alidade_description)/urdf/generated/alidade_${revision}.urdf"/>
+  <!-- Camera Intel D435i. Sa geometrie interne vient du paquet du constructeur,
+       qui est la source amont : on n'y accroche que notre point de fixation.
+       `use_nominal_extrinsics` decide qui publie les reperes optiques : en
+       simulation personne d'autre ne le fera, sur le robot c'est le driver, et
+       avec les extrinseques CALIBREES de l'exemplaire, que les nominales ne
+       feraient qu'approcher. -->
+  <xacro:property name="cam" value="${hw['camera']}"/>
+  <xacro:include filename="$(find realsense2_description)/urdf/_d435i.urdf.xacro"/>
+  <xacro:sensor_d435i parent="${cam['mount_link']}" name="${cam['name']}"
+                      use_nominal_extrinsics="${target == 'sim'}" use_mesh="false">
+    <origin xyz="${cam['mount_offset'][0]} ${cam['mount_offset'][1]} ${cam['mount_offset'][2]}"
+            rpy="0 0 0"/>
+  </xacro:sensor_d435i>
   <xacro:include filename="$(find alidade_description)/urdf/ros2_control.xacro"/>
   <xacro:alidade_ros2_control hw="${hw}" target="${target}" use_mock="${use_mock}" pico_port="$(arg pico_port)"/>

File: alidade_description/urdf/gazebo.xacro (robot description, xacro)
@@ -71,6 +71,10 @@
     <gazebo reference="${camera['frame']}">
       <sensor name="camera" type="camera">
-        <!-- gz publie l'image sur ce topic et le camera_info a cote de lui. -->
-        <topic>camera/image_raw</topic>
+        <!-- gz publie l'image sur ce topic et le camera_info a cote de lui.
+             Meme nom que le vrai pilote RealSense, pour qu'aruco_opencv et le
+             detecteur ne sachent pas de quel cote ils tournent. Seule la
+             COULEUR est simulee : la profondeur du D435i n'est encore utilisee
+             par rien, et un capteur rgbd en rendu logiciel coute cher. -->
+        <topic>camera/color/image_raw</topic>
         <update_rate>${camera['fps']}</update_rate>
         <always_on>1</always_on>

File: alidade_description/urdf/onshape/alidade_v2.urdf (robot description, URDF)
Before this commit: robot main_assembly, 26 links, 25 joints
Links:
- removed link camera_link
- removed link camera_optical_frame
- removed link caster_fork_link
- removed link caster_mount_link
- link base_link: mass 0.000109733 -> 0.000275747; geometry visual mesh filename=package://alidade_v2/meshes/base_link.stl scale=1 1 1
- link battery_link: geometry visual mesh filename=package://alidade_v2/meshes/battery_link.stl scale=1 1 1
- link battery_tray_link: geometry visual mesh filename=package://alidade_v2/meshes/battery_tray_link.stl scale=1 1 1
- link camera_mount_link: mass 1.31479e-05 -> 3.8641e-05; geometry visual mesh filename=package://alidade_v2/meshes/camera_mount_link.stl scale=1 1 1
- link caster_wheel_link: mass 5.57528e-06 -> 5.01392e-05; geometry visual mesh filename=package://alidade_v2/meshes/caster_wheel_link.stl scale=1 1 1
- link dcdc_link: geometry visual mesh filename=package://alidade_v2/meshes/dcdc_link.stl scale=1 1 1
- link deck_link: mass 7.67011e-05 -> 0.00014731; geometry visual mesh filename=package://alidade_v2/meshes/deck_link.stl scale=1 1 1
- link driver_board_link: geometry visual mesh filename=package://alidade_v2/meshes/driver_board_link.stl scale=1 1 1
- link imu_link: geometry visual mesh filename=package://alidade_v2/meshes/imu_link.stl scale=1 1 1
- link laser: geometry visual mesh filename=package://alidade_v2/meshes/laser.stl scale=1 1 1
- link motor_driver_left_link: geometry visual mesh filename=package://alidade_v2/meshes/motor_driver_left_link.stl scale=1 1 1
- link motor_driver_right_link: geometry visual mesh filename=package://alidade_v2/meshes/motor_driver_right_link.stl scale=1 1 1
- link motor_left_link: geometry visual mesh filename=package://alidade_v2/meshes/motor_left_link.stl scale=1 1 1
- link motor_mount_left_link: geometry visual mesh filename=package://alidade_v2/meshes/motor_mount_left_link.stl scale=1 1 1
- link motor_mount_right_link: geometry visual mesh filename=package://alidade_v2/meshes/motor_mount_right_link.stl scale=1 1 1
- link motor_right_link: geometry visual mesh filename=package://alidade_v2/meshes/motor_right_link.stl scale=1 1 1
- link pi_link: geometry visual mesh filename=package://alidade_v2/meshes/pi_link.stl scale=1 1 1
- link pi_mount_link: geometry visual mesh filename=package://alidade_v2/meshes/pi_mount_link.stl scale=1 1 1
- link power_bracket_link: geometry visual mesh filename=package://alidade_v2/meshes/power_bracket_link.stl scale=1 1 1
- link wheel_left_link: mass 3.20155e-05 -> 0.000167891; geometry visual mesh filename=package://alidade_v2/meshes/wheel_left_link.stl scale=1 1 1
- link wheel_right_link: mass 3.20155e-05 -> 0.000167891; geometry visual mesh filename=package://alidade_v2/meshes/wheel_right_link.stl scale=1 1 1
Joints:
- removed joint camera_joint
- removed joint camera_optical_frame
- removed joint caster_fork_joint
- removed joint caster_mount_joint
- joint base_joint: origin xyz=-0.038146 0 0.053104 rpy=0 -0 0 -> xyz=0.052 0 0.070601 rpy=-2.66454e-15 -2.66241e-30 1.77494e-30
- joint battery_joint: origin xyz=-0.0306365 5.51219e-11 0.005 rpy=-3.14159 -2.1684e-19 -6.66134e-16 -> xyz=-0.0306365 5.51219e-11 0.005 rpy=-3.14159 -2.1684e-19 -3.21271e-15
- joint battery_tray_joint: origin xyz=0.0717888 0 0.005 rpy=-1.33227e-15 1.33227e-15 7.21645e-16 -> xyz=-0.153984 -3.0166e-17 0.005 rpy=-2.66454e-15 3.65464e-30 -7.88861e-31
- joint camera_mount_joint: axis 0.34202 -0 -0.939693 -> -6.12323e-17 1.45363e-17 1; origin xyz=-0.0257 0.065 0.005 rpy=0 0.349066 0 -> xyz=-0.04 -1.2326e-32 0.045 rpy=1.45363e-17 6.12323e-17 4.45045e-34; parent deck_link -> base_link
- joint caster_wheel_joint: axis 0 0 1 -> -0 -0 1; origin xyz=0 0 3.46945e-18 rpy=-4.71845e-16 3.99823e-31 3.88578e-16 -> xyz=-0.24075 0.01875 0 rpy=-4.6598e-91 1.75162e-46 -5.32056e-45; parent caster_fork_link -> base_link
- joint dcdc_joint: origin xyz=-0.02335 -0.01345 0.005 rpy=0 -0 0 -> xyz=-0.02335 -0.01345 -0.0155 rpy=5.55112e-17 -5.55112e-17 5.55112e-17
- joint deck_joint: origin xyz=0.15015 -0.05 0.065 rpy=0 -0 0 -> xyz=-0.1225 0.0475 0.005 rpy=-5.32907e-15 1.06496e-29 -3.9443e-31
- joint driver_board_joint: axis -0 1 -0 -> 0 0 1; origin xyz=0.081575 -0.078 0 rpy=-5.55112e-16 3.33067e-16 6.12323e-17 -> xyz=-0.111954 -1.68498e-18 0 rpy=-2.66454e-15 2.66454e-15 1.5708
- joint imu_joint: origin xyz=-0.112165 0.05 0.01075 rpy=0 -0 0 -> xyz=-0.0539 -0.0026 -0.00457 rpy=-3.14159 -2.66241e-29 9.86076e-31; parent deck_link -> base_link
- joint laser_joint: origin xyz=-0.0664496 0.05 0.035596 rpy=1.40166e-15 -1.38778e-17 0 -> xyz=-0.0293 -0.0475 0.0895963 rpy=9.39526e-15 -1.38778e-17 5.25962e-30
- joint motor_driver_left_joint: origin xyz=0.01924 0.0156 -0.007 rpy=1.5708 4.996e-16 -1.5708 -> xyz=0.01924 -0.00941 -0.005 rpy=1.5708 5.55112e-17 -1.5708
- joint motor_driver_right_joint: origin xyz=-0.01924 0.0156 -0.007 rpy=1.5708 4.44089e-16 -1.5708 -> xyz=-0.01924 -0.00941 -0.005 rpy=1.5708 5.55112e-17 -1.5708
- joint motor_left_joint: origin xyz=-0.00815 0.00745 0.0206 rpy=1.5708 -5.55112e-16 3.14159 -> xyz=0.00815 0.00745 0.0206 rpy=1.5708 -1.19349e-15 3.14159
- joint motor_mount_left_joint: origin xyz=0.03 0.06755 0 rpy=-3.14159 2.05486e-16 3.14159 -> xyz=-0.04385 0.08955 1.38778e-17 rpy=3.14159 -8.09407e-28 3.14159
- joint motor_mount_right_joint: axis 0 0 -1 -> -0 -0 -1; origin xyz=0.03 -0.06755 0 rpy=3.14159 -4.05018e-16 1.94289e-16 -> xyz=-0.04385 -0.08955 1.38778e-17 rpy=-3.14159 4.16001e-32 -7.49401e-16
- joint motor_right_joint: origin xyz=0.00815 0.00745 0.0206 rpy=-1.5708 -2.498e-16 -1.17882e-16 -> xyz=-0.00815 0.00745 0.0206 rpy=-1.5708 -2.498e-16 3.81718e-16
- joint pi_joint: origin xyz=-0.0390428 0.0035 0.007 rpy=6.51193e-16 -9.51968e-18 -5.20656e-17 -> xyz=-0.0290428 -0.0245 0.007 rpy=-7.81319e-15 1.9984e-15 -1.249e-16
- joint pi_mount_joint: axis -0 -0 -1 -> 0 0 -1; origin xyz=0.15815 1.99493e-17 0.005 rpy=-1.69318e-16 3.61723e-16 1.5708 -> xyz=-0.0875 0.0025 0.0295 rpy=-1.5708 9.86076e-31 -1.77494e-30; parent base_link -> deck_link
- joint power_bracket_joint: origin xyz=0.094575 0.063 0 rpy=1.5708 -0 0 -> xyz=-0.136954 0.08 0 rpy=1.5708 4.71845e-15 1.5708
- joint wheel_left_joint: axis 0 -1 0 -> 0 1 0; origin xyz=-0.000128278 6.29059e-08 0.0205 rpy=-1.5708 -8.30461e-31 3.14159 -> xyz=4.03494e-06 4.21546e-08 0.0155 rpy=1.5708 3.33067e-16 6.245e-16
- joint wheel_right_joint: origin xyz=-0.000132313 2.07513e-08 0.0205 rpy=-1.5708 2.18632e-30 -1.64402e-17 -> xyz=1.00466e-20 6.93889e-18 0.0155 rpy=-1.5708 -5.27356e-16 8.32667e-17
