Commit message: description : nouveaux supports de camera et de LiDAR, export Onshape allege
Nouvel export de la CAO. Le LiDAR est abaisse de 26 mm et recule de 25 mm,
son support et celui de l'IMU sont fondus dans le plateau ; la camera, sur
un nouveau support, plonge de 25 degres. Les poses attendues de la revision
suivent, et fix_urdf les retrouve a 0.13 mm pres. Aucune piece ne coupe le
plan du LiDAR : la plus haute apres lui culmine a 130 mm, contre 153.7 mm
pour son repere.

Maillages exportes en resolution grossiere : 16 Mo au lieu des 116 Mo d'un
export fin. Le README note la marche a suivre apres un export, qui vide le
dossier urdf/.

File: alidade_description/urdf/onshape/alidade.urdf (robot description, URDF)
Before this commit: robot main_assembly, 27 links, 26 joints
Links:
- removed link imu_bracket_link
- removed link lidar_mount_link
- added link camera_mount_link, mass 1.30653e-05; visual mesh filename=package://main_assembly/meshes/camera_mount_link.stl scale=1 1 1
- link camera_link: mass 8.358e-05 -> 4.24237e-05
- link dcdc_link: mass 6.14564e-06 -> 8.34806e-06
- link deck_link: mass 0.000109733 -> 7.67011e-05
- link power_bracket_link: mass 6.48807e-06 -> 1.64647e-05
Joints:
- removed joint imu_bracket_joint
- removed joint lidar_mount_joint
- added joint camera_mount_joint: type fixed, parent deck_link, child camera_mount_link, origin xyz=-0.0257 0.065 0.005 rpy=0 0.436332 0, axis 0.422618 -0 -0.906308
- joint camera_joint: axis 6.12323e-17 6.12323e-17 -1 -> -6.12323e-17 1.2326e-32 1; origin xyz=0.0649646 0.0297332 0.021 rpy=8.81451e-16 -6.01243e-15 -1.77636e-15 -> xyz=0.0144098 -0.015 0.00901324 rpy=1.2326e-32 -3.00315e-07 0; parent lidar_mount_link -> camera_mount_link
- joint camera_optical_frame: origin xyz=0.0375 3.63822e-18 -0.0295 rpy=-1.5708 -0 -1.5708 -> xyz=0.0208 -3.46945e-18 -0.015 rpy=-1.5708 5.55112e-17 -1.5708
- joint dcdc_joint: axis -0 -1 -0 -> 0 1 0; origin xyz=-0.000293589 0.003 4.3198e-05 rpy=-2.22045e-15 -8.63198e-15 -1.8977e-15 -> xyz=-0.02335 -0.01345 0.005 rpy=0 -0 0
- joint deck_joint: origin xyz=0.15015 -0.05 0.065 rpy=3.33067e-16 -3.33067e-16 5.54668e-32 -> xyz=0.15015 -0.05 0.065 rpy=0 -0 0
- joint imu_joint: origin xyz=-0.00814078 -0.053552 0.00857 rpy=6.66134e-16 1.66533e-15 -3.14159 -> xyz=-0.112165 0.05 0.01075 rpy=0 -0 0; parent imu_bracket_link -> deck_link
- joint laser_joint: origin xyz=0.0276573 0.0297332 0.0565965 rpy=9.73346e-16 -5.9923e-15 -2.52576e-15 -> xyz=-0.0664496 0.05 0.035596 rpy=1.40166e-15 -1.38778e-17 0; parent lidar_mount_link -> deck_link
- joint power_bracket_joint: axis 0 -1 0 -> 0 1 0; origin xyz=0.086575 0.063 0 rpy=-1.5708 1.04916e-14 -6.60583e-15 -> xyz=0.094575 0.063 0 rpy=1.5708 -0 0

Commit message: description : support camera a 20 degres
Nouvel export Onshape : le support passe de 25 a 20 degres (0.436 -> 0.349
rad), seul le repere optique bouge (2.1 mm, pivot autour du support). La
correction de -3.2 degres mesuree au cube valait pour l'ancien support ; elle
est retiree, l'inclinaison reelle du nouveau reste a mesurer.

File: alidade_description/urdf/onshape/alidade.urdf (robot description, URDF)
Before this commit: robot main_assembly, 26 links, 25 joints
Links:
- link camera_mount_link: mass 1.30653e-05 -> 1.31479e-05
Joints:
- joint camera_joint: origin xyz=0.0144098 -0.015 0.00901324 rpy=1.2326e-32 -3.00315e-07 0 -> xyz=0.0150907 -0.015 0.00762285 rpy=1.2326e-32 -3.00315e-07 3.26265e-55
- joint camera_mount_joint: axis 0.422618 -0 -0.906308 -> 0.34202 -0 -0.939693; origin xyz=-0.0257 0.065 0.005 rpy=0 0.436332 0 -> xyz=-0.0257 0.065 0.005 rpy=0 0.349066 0
- joint camera_optical_frame: origin xyz=0.0208 -3.46945e-18 -0.015 rpy=-1.5708 5.55112e-17 -1.5708 -> xyz=0.0208 -3.46945e-18 -0.015 rpy=-1.5708 -0 -1.5708
