Commit message: la camera existe : pilote installe, profils valides, montage mesure
Premier branchement du D435i, et trois choses sortent.

LE PILOTE N'ETAIT PAS INSTALLE. ros-jazzy-realsense2-camera manquait sur le
robot -- system/install.sh n'avait pas ete rejoue depuis son ajout a
apt-packages.txt. Le conteneur echouait sur « Could not find requested resource
in ament index », et comme camera.launch.py saute le conteneur quand aucune
camera n'est branchee, l'erreur etait invisible. Rien a changer dans le depot :
le paquet y etait deja declare.

LES PROFILS ETAIENT REFUSES EN SILENCE. camera.fps valait 15.0, la chaine
rendue valait « 640x480x15.0 », et le pilote exige un entier : il se rabattait
sur 1280x720x30 en couleur et 848x480x30 en profondeur, soit 83 Mo/s au lieu de
13.8 sur un Pi 5. Le commentaire de la revision justifiait ce flottant a tort --
les deux autres consommateurs font float(hz) et <update_rate>. Passe en entier,
verifie : « Open profile: Color, 640x480, FPS: 15 ».

RE-EXPORT CAO recale sur le robot physique (merci), reporte dans la revision :
un maillon camera_adaptor s'intercale, camera_mount_link recule de 43.5 mm et
monte de 25.0 mm (ecart 50.17 mm), et le LiDAR monte de 9.0 mm. Les deux
rotations de pi de l'adaptateur s'annulent : pas d'inclinaison. footprint.height
suit le LiDAR, 0.1849.

Le x du laser ne bouge pas, donc tout le travail d'azimut du LiDAR reste valide.

camera.mount_link N'EST PLUS PROVISOIRE. Verifie en ajustant le plan du SOL sur
l'image de profondeur et en le ramenant dans base_link par TF, RANSAC contraint
en orientation seulement :

  hauteur du centre optique    152.6 mm mesures contre 153.1 modeles   -0.5 mm
  plan du sol                  +1.3 mm du z attendu
  inclinaison du montage       0.68 deg
  un mur, camera contre LiDAR  -1.3 mm (-0.20 %) et 0.42 deg

17 000 inliers de part et d'autre, residus 1.5 et 2.2 mm, deux capteurs
independants concordants. Et cette mesure avait DETECTE l'erreur avant la
correction CAO : elle annoncait la camera 19 a 31 mm trop haute, le re-export en
a releve 25.0.

250 tests, 0 echec. aruco_tracker detecte deja des marqueurs.

Co-Authored-By: Claude Opus 5 <noreply@anthropic.com>

File: alidade_description/urdf/onshape/alidade_v2.urdf (robot description, URDF)
Before this commit: robot alidade_v2, 22 links, 21 joints
Links:
- added link camera_adaptor, mass 2.69817e-05; visual mesh filename=package://alidade_v2/meshes/camera_adaptor.stl scale=1 1 1
Joints:
- added joint camera_adaptor_joint: type fixed, parent base_link, child camera_adaptor, origin xyz=-0.066 -0.06 0.065 rpy=-7.99361e-15 2.66454e-15 3.14159, axis 0 0 1
- joint base_joint: origin xyz=0.052 0 0.070601 rpy=-2.66454e-15 -2.66241e-30 1.77494e-30 -> xyz=0.052 0 0.070601 rpy=-7.99361e-15 5.45793e-29 3.9968e-15
- joint battery_tray_joint: origin xyz=-0.153984 -3.0166e-17 0.005 rpy=-2.66454e-15 3.65464e-30 -7.88861e-31 -> xyz=-0.153984 -2.41044e-18 0.005 rpy=2.66454e-15 -2.55579e-29 -3.9968e-15
- joint camera_mount_joint: origin xyz=-0.04 -1.2326e-32 0.045 rpy=1.45363e-17 6.12323e-17 4.45045e-34 -> xyz=0.0175 -0.06 0.005 rpy=1.45363e-17 6.12323e-17 -3.14159; parent base_link -> camera_adaptor
- joint caster_wheel_joint: origin xyz=-0.24075 0.01875 0 rpy=-4.6598e-91 1.75162e-46 -5.32056e-45 -> xyz=-0.24075 0.01875 0 rpy=5.32907e-15 -3.06177e-29 -3.9968e-15
- joint deck_joint: origin xyz=-0.1225 0.0475 0.005 rpy=-5.32907e-15 1.06496e-29 -3.9443e-31 -> xyz=-0.1225 0.0475 0.005 rpy=1.97215e-31 -3.06177e-29 -3.9968e-15
- joint driver_board_joint: origin xyz=-0.111954 -1.68498e-18 0 rpy=-2.66454e-15 2.66454e-15 1.5708 -> xyz=-0.111954 -5.15443e-18 0 rpy=-7.99361e-15 7.99361e-15 1.5708
- joint imu_joint: origin xyz=-0.0539 -0.0026 -0.00457 rpy=-3.14159 -2.66241e-29 9.86076e-31 -> xyz=-0.0539 -0.0026 -0.00457 rpy=-3.14159 -6.25665e-29 -3.9968e-15
- joint laser_joint: origin xyz=-0.0293 -0.0475 0.0895963 rpy=9.39526e-15 -1.38778e-17 5.25962e-30 -> xyz=-0.0293 -0.0475 0.0985963 rpy=1.40166e-15 -1.38778e-17 -9.72595e-33
- joint motor_driver_left_joint: origin xyz=0.01924 -0.00941 -0.005 rpy=1.5708 5.55112e-17 -1.5708 -> xyz=0.01924 -0.00941 -0.005 rpy=1.5708 -0 -1.5708
- joint motor_driver_right_joint: origin xyz=-0.01924 -0.00941 -0.005 rpy=1.5708 5.55112e-17 -1.5708 -> xyz=-0.01924 -0.00941 -0.005 rpy=1.5708 -0 -1.5708
- joint motor_mount_left_joint: origin xyz=-0.04385 0.08955 1.38778e-17 rpy=3.14159 -8.09407e-28 3.14159 -> xyz=-0.04385 0.08955 9.71445e-16 rpy=3.14159 -7.79529e-28 3.14159
- joint motor_mount_right_joint: origin xyz=-0.04385 -0.08955 1.38778e-17 rpy=-3.14159 4.16001e-32 -7.49401e-16 -> xyz=-0.04385 -0.08955 -9.4369e-16 rpy=-3.14159 -3.19073e-29 -4.7462e-15
- joint power_bracket_joint: origin xyz=-0.136954 0.08 0 rpy=1.5708 4.71845e-15 1.5708 -> xyz=-0.136954 0.08 0 rpy=1.5708 1.40443e-14 1.5708
